File: HARDWARE/EDA/KICAD/PLC/PLC.kicad_pcb (KiCad board)
At the start: 2 copper layers, 555.2 x 225.5 mm, 207 parts, among them J2 retified-output, J3 power

Commit message: project in pcb
Parts:
- added D10: LED 3V, LED_THT:LED_D5.0mm_Clear, F.Cu at (386.0, 96.8)
- added D11: LED 3V, LED_THT:LED_D5.0mm_Clear, F.Cu at (398.2, 96.8)
- added D12: LED 3V, LED_THT:LED_D5.0mm_Clear, F.Cu at (410.2, 96.8)
- added D13: LED 3V, LED_THT:LED_D5.0mm_Clear, F.Cu at (422.2, 96.8)
- added D14: LED 3V, LED_THT:LED_D5.0mm_Clear, F.Cu at (434.2, 96.8)
- added D15: LED 3V, LED_THT:LED_D5.0mm_Clear, F.Cu at (446.8, 96.8)
- added D16: LED 3V, LED_THT:LED_D5.0mm_Clear, F.Cu at (460.8, 96.8)
- added D18: LED 3V, LED_THT:LED_D5.0mm_Clear, F.Cu at (449.2, 58.5)
- added D19: LED 3V, LED_THT:LED_D5.0mm_Clear, F.Cu at (436.8, 58.5)
- added D20: LED 3V, LED_THT:LED_D5.0mm_Clear, F.Cu at (424.8, 58.5)
- added D21: LED 3V, LED_THT:LED_D5.0mm_Clear, F.Cu at (412.8, 58.5)
- added D22: LED 3V, LED_THT:LED_D5.0mm_Clear, F.Cu at (400.8, 58.5)
- added D23: LED 3V, LED_THT:LED_D5.0mm_Clear, F.Cu at (386.0, 70.5)
- added D24: LED 3V, LED_THT:LED_D5.0mm_Clear, F.Cu at (398.2, 70.5)
- added D25: LED 3V, LED_THT:LED_D5.0mm_Clear, F.Cu at (410.2, 70.5)
- added D26: LED 3V, LED_THT:LED_D5.0mm_Clear, F.Cu at (422.2, 70.5)
- added D27: LED 3V, LED_THT:LED_D5.0mm_Clear, F.Cu at (434.2, 70.5)
- added D28: LED 3V, LED_THT:LED_D5.0mm_Clear, F.Cu at (446.8, 70.5)
- added D29: LED 3V, LED_THT:LED_D5.0mm_Clear, F.Cu at (460.8, 70.5)
- added D30: LED 3V, LED_THT:LED_D5.0mm_Clear, F.Cu at (463.2, 83.0)
- added D31: LED 3V, LED_THT:LED_D5.0mm_Clear, F.Cu at (434.2, 22.8)
- added D32: LED 3V, LED_THT:LED_D5.0mm_Clear, F.Cu at (446.8, 22.8)
- added D33: LED 3V, LED_THT:LED_D5.0mm_Clear, F.Cu at (460.8, 22.8)
- added D34: LED 3V, LED_THT:LED_D5.0mm_Clear, F.Cu at (463.2, 34.2)
- added D35: LED 3V, LED_THT:LED_D5.0mm_Clear, F.Cu at (449.2, 34.2)
- added D36: LED 3V, LED_THT:LED_D5.0mm_Clear, F.Cu at (436.8, 34.2)
- added D37: LED 3V, LED_THT:LED_D5.0mm_Clear, F.Cu at (424.8, 34.2)
- added D38: LED 3V, LED_THT:LED_D5.0mm_Clear, F.Cu at (410.2, 46.5)
- added D39: LED 3V, LED_THT:LED_D5.0mm_Clear, F.Cu at (422.2, 46.5)
- added D4: LED 3V, LED_THT:LED_D5.0mm_Clear, F.Cu at (449.2, 83.0)
- added D40: LED 3V, LED_THT:LED_D5.0mm_Clear, F.Cu at (434.2, 46.5)
- added D41: LED 3V, LED_THT:LED_D5.0mm_Clear, F.Cu at (446.8, 46.5)
- added D42: LED 3V, LED_THT:LED_D5.0mm_Clear, F.Cu at (460.8, 46.5)
- added D43: LED 3V, LED_THT:LED_D5.0mm_Clear, F.Cu at (463.2, 58.5)
- added D5: LED 3V, LED_THT:LED_D5.0mm_Clear, F.Cu at (436.8, 83.0)
- added D6: LED 3V, LED_THT:LED_D5.0mm_Clear, F.Cu at (424.8, 83.0)
- added D7: LED 3V, LED_THT:LED_D5.0mm_Clear, F.Cu at (412.8, 83.0)
- added D8: LED 3V, LED_THT:LED_D5.0mm_Clear, F.Cu at (400.8, 83.0)
- added D9: LED 3V, LED_THT:LED_D5.0mm_Clear, F.Cu at (388.5, 83.0)
Other:
- board size 555.2 x 225.5 mm -> 849.5 x 225.5 mm

Commit message: adjust pcb
Parts:
- removed the D10 at (386.0, 96.8)
- removed the D10 at (-263.0, 72.8)
- removed the D11 at (398.2, 96.8)
- removed the D11 at (-250.8, 72.8)
- removed the D12 at (410.2, 96.8)
- removed the D12 at (-238.8, 72.8)
- removed the D13 at (422.2, 96.8)
- removed the D13 at (-226.8, 72.8)
- removed the D14 at (434.2, 96.8)
- removed the D14 at (-214.8, 72.8)
- removed the D15 at (446.8, 96.8)
- removed the D15 at (-202.2, 72.8)
- removed the D16 at (460.8, 96.8)
- removed the D16 at (-188.2, 72.8)
- removed the D18 at (449.2, 58.5)
- removed the D18 at (-199.8, 34.5)
- removed the D19 at (436.8, 58.5)
- removed the D19 at (-212.2, 34.5)
- removed the D20 at (424.8, 58.5)
- removed the D20 at (-224.2, 34.5)
- removed the D21 at (412.8, 58.5)
- removed the D21 at (-236.2, 34.5)
- removed the D22 at (400.8, 58.5)
- removed the D22 at (-248.2, 34.5)
- removed the D23 at (386.0, 70.5)
- removed the D23 at (-263.0, 46.5)
- removed the D24 at (398.2, 70.5)
- removed the D24 at (-250.8, 46.5)
- removed the D25 at (410.2, 70.5)
- removed the D25 at (-238.8, 46.5)
- removed the D26 at (422.2, 70.5)
- removed the D26 at (-226.8, 46.5)
- removed the D27 at (434.2, 70.5)
- removed the D27 at (-214.8, 46.5)
- removed the D28 at (446.8, 70.5)
- removed the D28 at (-202.2, 46.5)
- removed the D29 at (460.8, 70.5)
- removed the D29 at (-188.2, 46.5)
- removed the D30 at (463.2, 83.0)
- removed the D30 at (-185.8, 59.0)
- removed the D31 at (434.2, 22.8)
- removed the D31 at (-214.8, -1.25)
- removed the D32 at (446.8, 22.8)
- removed the D32 at (-202.2, -1.25)
- removed the D33 at (460.8, 22.8)
- removed the D33 at (-188.2, -1.25)
- removed the D34 at (463.2, 34.2)
- removed the D34 at (-185.8, 10.2)
- removed the D35 at (449.2, 34.2)
- removed the D35 at (-199.8, 10.2)
- removed the D36 at (436.8, 34.2)
- removed the D36 at (-212.2, 10.2)
- removed the D37 at (424.8, 34.2)
- removed the D37 at (-224.2, 10.2)
- removed the D38 at (410.2, 46.5)
- removed the D38 at (-238.8, 22.5)
- removed the D39 at (422.2, 46.5)
- removed the D39 at (-226.8, 22.5)
- removed the D4 at (449.2, 83.0)
- removed the D4 at (-199.8, 59.0)
- removed the D40 at (434.2, 46.5)
- removed the D40 at (-214.8, 22.5)
- removed the D41 at (446.8, 46.5)
- removed the D41 at (-202.2, 22.5)
- removed the D42 at (460.8, 46.5)
- removed the D42 at (-188.2, 22.5)
- removed the D43 at (463.2, 58.5)
- removed the D43 at (-185.8, 34.5)
- removed the D5 at (436.8, 83.0)
- removed the D5 at (-212.2, 59.0)
- removed the D6 at (424.8, 83.0)
- removed the D6 at (-224.2, 59.0)
- removed the D7 at (412.8, 83.0)
- removed the D7 at (-236.2, 59.0)
- removed the D8 at (400.8, 83.0)
- removed the D8 at (-248.2, 59.0)
- removed the D9 at (388.5, 83.0)
- removed the D9 at (-260.5, 59.0)
Other:
- board size 849.5 x 225.5 mm -> 565.2 x 201.2 mm
- board text added: "15º, 20º, 30º, 60º, 0º"
- board text added: "24+18+12+6+1 = 61 LEDS"
- board text added: "ALIMENTAÇÃO DE 12 V 15 SÉRIES DE 4 LEDS 1 SÉRIE DE 1 LED COM 1 RESISTOR TOTAL 61 LEDS e um resistor resistor = 430 Ohms"

Commit message: reorganized schematic
Parts:
- removed C1: 250V, Capacitor_THT:CP_Radial_D18.0mm_P7.50mm
- removed the D1 at (248.5, 48.4)
- removed the D10 at (21.0, 97.8)
- removed D100, D101, D102, D103, D104, D105, D106, D107, D108, D109, D110, D111, D112, D113, D114, D115, D116, D117, D118, D119, D120, D121, D83, D84, D85, D86, D87, D88, D89, D90, D91, D92, D93, D94, D95, D96, D97, D98, D99: LED 3V, LED_THT:LED_D5.0mm_Clear
- removed the D11 at (33.2, 97.8)
- removed the D12 at (45.2, 97.8)
- removed D122, D123, D124, D125, D126, D127, D128, D129, D130, D131, D132, D133, D134, D135, D136, D137, D138, D139, D140, D141, D142, D143, D144, D145, D146, D147, D148, D149, D150, D151, D152, D153, D154, D155, D156, D157, D158, D159, D160, D62, D63, D64, D65, D66, D67, D68, D69, D70, D71, D72, D73, D74, D75, D76, D77, D78, D79, D80, D81, D82: LED 3V, LED_THT:LED_D5.0mm
- removed the D13 at (57.2, 97.8)
- removed the D14 at (69.2, 97.8)
- removed the D15 at (81.8, 97.8)
- removed the D16 at (95.8, 97.8)
- removed the D17 at (251.9, 38.5)
- removed the D18 at (84.2, 59.5)
- removed the D19 at (71.8, 59.5)
- removed the D2 at (245.0, 38.4)
- removed the D20 at (59.8, 59.5)
- removed the D21 at (47.8, 59.5)
- removed the D22 at (35.8, 59.5)
- removed the D23 at (21.0, 71.5)
- removed the D24 at (33.2, 71.5)
- removed the D25 at (45.2, 71.5)
- removed the D26 at (57.2, 71.5)
- removed the D27 at (69.2, 71.5)
- removed the D28 at (81.8, 71.5)
- removed the D29 at (95.8, 71.5)
- removed the D3 at (255.4, 48.5)
- removed the D30 at (98.2, 84.0)
- removed the D31 at (69.2, 23.8)
- removed the D32 at (81.8, 23.8)
- removed the D33 at (95.8, 23.8)
- removed the D34 at (98.2, 35.2)
- removed the D35 at (84.2, 35.2)
- removed the D36 at (71.8, 35.2)
- removed the D37 at (59.8, 35.2)
- removed the D38 at (45.2, 47.5)
- removed the D39 at (57.2, 47.5)
- removed the D4 at (84.2, 84.0)
- removed the D40 at (69.2, 47.5)
- removed the D41 at (81.8, 47.5)
- removed the D42 at (95.8, 47.5)
- removed the D43 at (98.2, 59.5)
- removed the D44 at (83.0, 124.5)
- removed the D45 at (83.0, 137.2)
- removed the D46 at (83.0, 149.2)
- removed the D47 at (83.0, 161.2)
- removed the D48 at (83.0, 173.5)
- removed the D49 at (83.0, 185.0)
- removed the D5 at (71.8, 84.0)
- removed the D50 at (97.0, 187.5)
- removed the D51 at (97.0, 176.0)
- removed the D52 at (97.0, 163.8)
- removed the D53 at (97.0, 151.8)
- removed the D54 at (97.0, 139.8)
- removed the D55 at (97.0, 127.0)
- removed the D56 at (97.0, 113.5)
- removed the D57 at (58.5, 124.5)
- removed the D58 at (58.5, 137.2)
- removed the D59 at (58.5, 149.2)
- removed the D6 at (59.8, 84.0)
- removed the D60 at (58.5, 161.2)
- removed the D61 at (58.5, 173.5)
- removed the D7 at (47.8, 84.0)
- removed the D8 at (35.8, 84.0)
- removed the D9 at (23.5, 84.0)
- removed F1, F2: Fuse, Fuse:Fuse_Blade_ATO_directSolder
- removed J2: retified-output, Connector_Phoenix_MC_HighVoltage:PhoenixContact_MC_1,5_2-G-5.08_1x02_P5.08mm_Horizontal
- removed J3: power, Connector_Phoenix_MC_HighVoltage:PhoenixContact_MC_1,5_3-G-5.08_1x03_P5.08mm_Horizontal
- removed RV1, RV2, RV3: Varistor 250V, Varistor:RV_Disc_D12mm_W4mm_P7.5mm
- added D1: LED, LED_THT:LED_D5.0mm, F.Cu at (469.8, -237.8)
- added D1: LED, LED_THT:LED_D5.0mm, F.Cu at (634.0, -322.0)
- added D1: LED, LED_THT:LED_D5.0mm, F.Cu at (433.3, 83.3)
- added D10: LED, LED_THT:LED_D5.0mm_IRBlack, F.Cu at (627.0, -304.0)
- added D10: LED, LED_THT:LED_D5.0mm_IRBlack, F.Cu at (469.0, 62.7)
- added D11: LED, LED_THT:LED_D5.0mm_IRBlack, F.Cu at (620.0, -304.0)
- added D11: LED, LED_THT:LED_D5.0mm_IRBlack, F.Cu at (458.4, 43.7)
- added D12: LED, LED_THT:LED_D5.0mm_IRBlack, F.Cu at (613.0, -304.0)
- added D12: LED, LED_THT:LED_D5.0mm_IRBlack, F.Cu at (448.0, 25.5)
- added D13: LED, LED_THT:LED_D5.0mm_IRGrey, F.Cu at (634.0, -295.0)
- added D13: LED, LED_THT:LED_D5.0mm_IRGrey, F.Cu at (479.6, 122.4)
- added D14: LED, LED_THT:LED_D5.0mm_IRGrey, F.Cu at (627.0, -295.0)
- added D14: LED, LED_THT:LED_D5.0mm_IRGrey, F.Cu at (489.6, 139.7)
- added D15: LED, LED_THT:LED_D5.0mm_IRGrey, F.Cu at (620.0, -295.0)
- added D15: LED, LED_THT:LED_D5.0mm_IRGrey, F.Cu at (499.6, 157.0)
- added D16: LED, LED_THT:LED_D5.0mm_IRGrey, F.Cu at (613.0, -295.0)
- added D16: LED, LED_THT:LED_D5.0mm_IRGrey, F.Cu at (509.6, 174.4)
- added D17: LED, LED_THT:LED_D5.0mm, F.Cu at (634.0, -286.0)
- added D17: LED, LED_THT:LED_D5.0mm, F.Cu at (458.4, 122.4)
- added D18: LED, LED_THT:LED_D5.0mm, F.Cu at (627.0, -286.0)
- added D18: LED, LED_THT:LED_D5.0mm, F.Cu at (448.4, 139.7)
- added D19: LED, LED_THT:LED_D5.0mm, F.Cu at (620.0, -286.0)
- added D19: LED, LED_THT:LED_D5.0mm, F.Cu at (438.4, 157.0)
- added D2: LED, LED_THT:LED_D5.0mm, F.Cu at (460.4, -256.2)
- added D2: LED, LED_THT:LED_D5.0mm, F.Cu at (627.0, -322.0)
- added D2: LED, LED_THT:LED_D5.0mm, F.Cu at (422.1, 64.6)
- added D20: LED, LED_THT:LED_D5.0mm, F.Cu at (613.0, -286.0)
- added D20: LED, LED_THT:LED_D5.0mm, F.Cu at (428.4, 174.4)
- added D21: LED, LED_THT:LED_D5.0mm_Clear, F.Cu at (634.0, -277.0)
- added D21: LED, LED_THT:LED_D5.0mm_Clear, F.Cu at (629.0, 80.0)
- added D22: LED, LED_THT:LED_D5.0mm_Clear, F.Cu at (627.0, -277.0)
- added D22: LED, LED_THT:LED_D5.0mm_Clear, F.Cu at (622.0, 80.0)
- added D23: LED, LED_THT:LED_D5.0mm_Clear, F.Cu at (620.0, -277.0)
- added D23: LED, LED_THT:LED_D5.0mm_Clear, F.Cu at (615.0, 80.0)
- added D24: LED, LED_THT:LED_D5.0mm_Clear, F.Cu at (613.0, -277.0)
- added D24: LED, LED_THT:LED_D5.0mm_Clear, F.Cu at (608.0, 80.0)
- added D25: LED, LED_THT:LED_D5.0mm_IRBlack, F.Cu at (634.0, -268.0)
- added D25: LED, LED_THT:LED_D5.0mm_IRBlack, F.Cu at (629.0, 89.0)
- added D26: LED, LED_THT:LED_D5.0mm_IRBlack, F.Cu at (627.0, -268.0)
- added D26: LED, LED_THT:LED_D5.0mm_IRBlack, F.Cu at (622.0, 89.0)
- added D27: LED, LED_THT:LED_D5.0mm_IRBlack, F.Cu at (620.0, -268.0)
- added D27: LED, LED_THT:LED_D5.0mm_IRBlack, F.Cu at (615.0, 89.0)
- added D28: LED, LED_THT:LED_D5.0mm_IRBlack, F.Cu at (613.0, -268.0)
- added D28: LED, LED_THT:LED_D5.0mm_IRBlack, F.Cu at (608.0, 89.0)
- added D29: LED, LED_THT:LED_D5.0mm_IRGrey, F.Cu at (634.0, -259.0)
- added D29: LED, LED_THT:LED_D5.0mm_IRGrey, F.Cu at (629.0, 98.0)
- added D3: LED, LED_THT:LED_D5.0mm, F.Cu at (481.6, -256.2)
- added D3: LED, LED_THT:LED_D5.0mm, F.Cu at (620.0, -322.0)
- added D3: LED, LED_THT:LED_D5.0mm, F.Cu at (411.5, 46.5)
- added D30: LED, LED_THT:LED_D5.0mm_IRGrey, F.Cu at (627.0, -259.0)
- added D30: LED, LED_THT:LED_D5.0mm_IRGrey, F.Cu at (622.0, 98.0)
- added D31: LED, LED_THT:LED_D5.0mm_IRGrey, F.Cu at (620.0, -259.0)
- added D31: LED, LED_THT:LED_D5.0mm_IRGrey, F.Cu at (615.0, 98.0)
- added D32: LED, LED_THT:LED_D5.0mm_IRGrey, F.Cu at (613.0, -259.0)
- added D32: LED, LED_THT:LED_D5.0mm_IRGrey, F.Cu at (608.0, 98.0)
- added D33: LED, LED_THT:LED_D5.0mm, F.Cu at (634.0, -250.0)
- added D33: LED, LED_THT:LED_D5.0mm, F.Cu at (629.0, 107.0)
- added D34: LED, LED_THT:LED_D5.0mm, F.Cu at (627.0, -250.0)
- added D34: LED, LED_THT:LED_D5.0mm, F.Cu at (622.0, 107.0)
- added D35: LED, LED_THT:LED_D5.0mm, F.Cu at (620.0, -250.0)
- added D35: LED, LED_THT:LED_D5.0mm, F.Cu at (615.0, 107.0)
- added D36: LED, LED_THT:LED_D5.0mm, F.Cu at (613.0, -250.0)
- added D36: LED, LED_THT:LED_D5.0mm, F.Cu at (608.0, 107.0)
- added D37: LED, LED_THT:LED_D5.0mm_Clear, F.Cu at (634.0, -241.0)
- added D37: LED, LED_THT:LED_D5.0mm_Clear, F.Cu at (629.0, 116.0)
- added D38: LED, LED_THT:LED_D5.0mm_Clear, F.Cu at (627.0, -241.0)
- added D38: LED, LED_THT:LED_D5.0mm_Clear, F.Cu at (622.0, 116.0)
- added D39: LED, LED_THT:LED_D5.0mm_Clear, F.Cu at (620.0, -241.0)
- added D39: LED, LED_THT:LED_D5.0mm_Clear, F.Cu at (615.0, 116.0)
- added D4: LED, LED_THT:LED_D5.0mm, F.Cu at (492.2, -237.8)
- added D4: LED, LED_THT:LED_D5.0mm, F.Cu at (613.0, -322.0)
- added D4: LED, LED_THT:LED_D5.0mm, F.Cu at (398.6, 63.4)
- added D40: LED, LED_THT:LED_D5.0mm_Clear, F.Cu at (613.0, -241.0)
- added D40: LED, LED_THT:LED_D5.0mm_Clear, F.Cu at (608.0, 116.0)
- added D41: LED, LED_THT:LED_D5.0mm_IRBlack, F.Cu at (634.0, -232.0)
- added D41: LED, LED_THT:LED_D5.0mm_IRBlack, F.Cu at (629.0, 125.0)
- added D42: LED, LED_THT:LED_D5.0mm_IRBlack, F.Cu at (627.0, -232.0)
- added D42: LED, LED_THT:LED_D5.0mm_IRBlack, F.Cu at (622.0, 125.0)
- added D43: LED, LED_THT:LED_D5.0mm_IRBlack, F.Cu at (620.0, -232.0)
- added D43: LED, LED_THT:LED_D5.0mm_IRBlack, F.Cu at (615.0, 125.0)
- added D44: LED, LED_THT:LED_D5.0mm_IRBlack, F.Cu at (613.0, -232.0)
- added D44: LED, LED_THT:LED_D5.0mm_IRBlack, F.Cu at (608.0, 125.0)
- added D45: LED, LED_THT:LED_D5.0mm_IRGrey, F.Cu at (634.0, -223.0)
- added D45: LED, LED_THT:LED_D5.0mm_IRGrey, F.Cu at (629.0, 134.0)
- added D46: LED, LED_THT:LED_D5.0mm_IRGrey, F.Cu at (627.0, -223.0)
- added D46: LED, LED_THT:LED_D5.0mm_IRGrey, F.Cu at (622.0, 134.0)
- added D47: LED, LED_THT:LED_D5.0mm_IRGrey, F.Cu at (620.0, -223.0)
- added D47: LED, LED_THT:LED_D5.0mm_IRGrey, F.Cu at (615.0, 134.0)
- added D48: LED, LED_THT:LED_D5.0mm_IRGrey, F.Cu at (613.0, -223.0)
- added D48: LED, LED_THT:LED_D5.0mm_IRGrey, F.Cu at (608.0, 134.0)
- added D49: LED, LED_THT:LED_D5.0mm, F.Cu at (634.0, -214.0)
- added D49: LED, LED_THT:LED_D5.0mm, F.Cu at (629.0, 143.0)
- added D5: LED, LED_THT:LED_D5.0mm_Clear, F.Cu at (634.0, -313.0)
- added D5: LED, LED_THT:LED_D5.0mm_Clear, F.Cu at (458.4, 85.6)
- added D50: LED, LED_THT:LED_D5.0mm, F.Cu at (627.0, -214.0)
- added D50: LED, LED_THT:LED_D5.0mm, F.Cu at (622.0, 143.0)
- added D51: LED, LED_THT:LED_D5.0mm, F.Cu at (620.0, -214.0)
- added D51: LED, LED_THT:LED_D5.0mm, F.Cu at (615.0, 143.0)
- added D52: LED, LED_THT:LED_D5.0mm, F.Cu at (613.0, -214.0)
- added D52: LED, LED_THT:LED_D5.0mm, F.Cu at (608.0, 143.0)
- added D53: LED, LED_THT:LED_D5.0mm_Clear, F.Cu at (634.0, -205.0)
- added D53: LED, LED_THT:LED_D5.0mm_Clear, F.Cu at (629.0, 152.0)
- added D54: LED, LED_THT:LED_D5.0mm_Clear, F.Cu at (627.0, -205.0)
- added D54: LED, LED_THT:LED_D5.0mm_Clear, F.Cu at (622.0, 152.0)
- added D55: LED, LED_THT:LED_D5.0mm_Clear, F.Cu at (620.0, -205.0)
- added D55: LED, LED_THT:LED_D5.0mm_Clear, F.Cu at (615.0, 152.0)
- added D56: LED, LED_THT:LED_D5.0mm_Clear, F.Cu at (613.0, -205.0)
- added D56: LED, LED_THT:LED_D5.0mm_Clear, F.Cu at (608.0, 152.0)
- added D57: LED, LED_THT:LED_D5.0mm_IRBlack, F.Cu at (634.0, -196.0)
- added D57: LED, LED_THT:LED_D5.0mm_IRBlack, F.Cu at (629.0, 161.0)
- added D58: LED, LED_THT:LED_D5.0mm_IRBlack, F.Cu at (627.0, -196.0)
- added D58: LED, LED_THT:LED_D5.0mm_IRBlack, F.Cu at (622.0, 161.0)
- added D59: LED, LED_THT:LED_D5.0mm_IRBlack, F.Cu at (620.0, -196.0)
- added D59: LED, LED_THT:LED_D5.0mm_IRBlack, F.Cu at (615.0, 161.0)
- added D6: LED, LED_THT:LED_D5.0mm_Clear, F.Cu at (627.0, -313.0)
- added D6: LED, LED_THT:LED_D5.0mm_Clear, F.Cu at (448.4, 68.3)
- added D60: LED, LED_THT:LED_D5.0mm_IRBlack, F.Cu at (613.0, -196.0)
- added D60: LED, LED_THT:LED_D5.0mm_IRBlack, F.Cu at (608.0, 161.0)
- added D61: LED, LED_THT:LED_D5.0mm_IRGrey, F.Cu at (634.0, -186.0)
- added D61: LED, LED_THT:LED_D5.0mm_IRGrey, F.Cu at (629.0, 171.0)
- added D7: LED, LED_THT:LED_D5.0mm_Clear, F.Cu at (620.0, -313.0)
- added D7: LED, LED_THT:LED_D5.0mm_Clear, F.Cu at (438.4, 51.0)
- added D8: LED, LED_THT:LED_D5.0mm_Clear, F.Cu at (613.0, -313.0)
- added D8: LED, LED_THT:LED_D5.0mm_Clear, F.Cu at (428.4, 33.6)
- added D9: LED, LED_THT:LED_D5.0mm_IRBlack, F.Cu at (634.0, -304.0)
- added D9: LED, LED_THT:LED_D5.0mm_IRBlack, F.Cu at (479.6, 85.6)
- added R1: 430 R, Resistor_THT:R_Axial_DIN0207_L6.3mm_D2.5mm_P7.62mm_Horizontal, F.Cu at (621.4, -186.0)
- added R1: 430 R, Resistor_THT:R_Axial_DIN0207_L6.3mm_D2.5mm_P7.62mm_Horizontal, F.Cu at (616.4, 171.0)
Routing:
- net GND: track 1401.9 -> 0.00 mm
- net GROUP1: track 1267.1 -> 0.00 mm
- net Net-(D22-Pad2): track 17.8 -> 0.00 mm
- net Net-(D61-Pad2): track 17.8 -> 0.00 mm
- net Net-(D100-Pad2): track 17.8 -> 0.00 mm
- net Net-(D139-Pad2): track 17.8 -> 0.00 mm
- net Net-(D127-Pad2): track 13.8 -> 0.00 mm
- net Net-(D88-Pad2): track 13.8 -> 0.00 mm
- net Net-(D49-Pad2): track 13.8 -> 0.00 mm
- net Net-(D10-Pad1): track 13.8 -> 0.00 mm
- net Net-(D146-Pad2): track 12.5 -> 0.00 mm
- net Net-(D107-Pad2): track 12.5 -> 0.00 mm
- net Net-(D68-Pad2): track 12.5 -> 0.00 mm
- net Net-(D29-Pad2): track 12.5 -> 0.00 mm
- net Net-(D42-Pad2): track 12.0 -> 0.00 mm
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Other:
- board size 565.2 x 201.2 mm -> 202 x 541.8 mm

Commit message: finished schematic and PCB
Parts:
- removed the D1 at (469.8, -237.8)
- removed the D1 at (433.3, 83.3)
- removed the D11 at (620.0, -304.0)
- removed the D11 at (458.4, 43.7)
- removed the D15 at (620.0, -295.0)
- removed the D15 at (499.6, 157.0)
- removed the D2 at (460.4, -256.2)
- removed the D2 at (422.1, 64.6)
- removed the D3 at (481.6, -256.2)
- removed the D3 at (411.5, 46.5)
- removed the D4 at (492.2, -237.8)
- removed the D4 at (398.6, 63.4)
- removed the R1 at (621.4, -186.0)
- removed the R1 at (616.4, 171.0)
- added D1: LED, LED_THT:LED_D5.0mm, F.Cu at (732.4, -326.9)
- added D11: LED, LED_THT:LED_D5.0mm_IRBlack, F.Cu at (718.4, -308.9)
- added D11: LED, LED_THT:LED_D5.0mm_IRBlack, F.Cu at (447.8, 69.4)
- added D15: LED, LED_THT:LED_D5.0mm_IRGrey, F.Cu at (718.4, -299.9)
- added D15: LED, LED_THT:LED_D5.0mm_IRGrey, F.Cu at (507.7, 104.0)
- added D2: LED, LED_THT:LED_D5.0mm, F.Cu at (725.4, -326.9)
- added D3: LED, LED_THT:LED_D5.0mm, F.Cu at (718.4, -326.9)
- added D4: LED, LED_THT:LED_D5.0mm, F.Cu at (711.4, -326.9)
- added R1: 430 R, Resistor_THT:R_Axial_DIN0207_L6.3mm_D2.5mm_P7.62mm_Horizontal, F.Cu at (719.8, -190.9)
- added R1: 430 R, Resistor_THT:R_Axial_DIN0207_L6.3mm_D2.5mm_P7.62mm_Horizontal, F.Cu at (416.8, 173.2)
- moved D20 544.6 mm to (711.4, -290.9), turned to 0 degrees
- moved D19 528.3 mm to (718.4, -290.9), turned to 0 degrees
- moved D16 515.4 mm to (711.4, -299.9), turned to 0 degrees
- moved D18 512.0 mm to (725.4, -290.9), turned to 0 degrees
- moved D14 498.9 mm to (725.4, -299.9), turned to 0 degrees
- moved D17 495.9 mm to (732.4, -290.9), turned to 0 degrees
- moved D13 492.2 mm to (732.4, -299.9), turned to 0 degrees
- moved D5 487.7 mm to (732.4, -317.9), turned to 0 degrees
- moved D6 475.3 mm to (725.4, -317.9), turned to 0 degrees
- moved D8 472.6 mm to (433.1, 124.0)
- moved D20 469.4 mm to (421.7, 142.6)
- moved D9 468.5 mm to (732.4, -308.9), turned to 0 degrees
- moved D7 463.7 mm to (457.7, 121.4)
- moved D7 463.1 mm to (718.4, -317.9), turned to 0 degrees
- moved D2 462.2 mm to (447.7, 104.0)
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Connections:
- D1 pad 1: (no net) -> Net-(D1-Pad1)
- D1 pad 2: (no net) -> +12V
- D10 pad 1: Net-(D10-Pad1) -> (no net)
- D10 pad 2: Net-(D10-Pad2) -> (no net)
- D10 pad 1: (no net) -> Net-(D10-Pad1)
- D10 pad 2: (no net) -> Net-(D10-Pad2)
- D12 pad 1: GND -> (no net)
- D12 pad 2: Net-(D11-Pad1) -> (no net)
- D12 pad 1: (no net) -> GND
- D12 pad 2: (no net) -> Net-(D11-Pad1)
- D13 pad 1: Net-(D13-Pad1) -> (no net)
- D13 pad 2: +12V -> (no net)
- D13 pad 1: (no net) -> Net-(D13-Pad1)
- D13 pad 2: (no net) -> +12V
- D14 pad 1: Net-(D14-Pad1) -> (no net)
- D14 pad 2: Net-(D13-Pad1) -> (no net)
- D14 pad 1: (no net) -> Net-(D14-Pad1)
- D14 pad 2: (no net) -> Net-(D13-Pad1)
- D16 pad 1: GND -> (no net)
- D16 pad 2: Net-(D15-Pad1) -> (no net)
- D16 pad 1: (no net) -> GND
- D16 pad 2: (no net) -> Net-(D15-Pad1)
- D17 pad 1: Net-(D17-Pad1) -> (no net)
- D17 pad 2: +12V -> (no net)
- D17 pad 1: (no net) -> Net-(D17-Pad1)
- D17 pad 2: (no net) -> +12V
- D18 pad 1: Net-(D18-Pad1) -> (no net)
- D18 pad 2: Net-(D17-Pad1) -> (no net)
- D18 pad 1: (no net) -> Net-(D18-Pad1)
- D18 pad 2: (no net) -> Net-(D17-Pad1)
- D19 pad 1: Net-(D19-Pad1) -> (no net)
- D19 pad 2: Net-(D18-Pad1) -> (no net)
- D19 pad 1: (no net) -> Net-(D19-Pad1)
- D19 pad 2: (no net) -> Net-(D18-Pad1)
- D2 pad 1: (no net) -> Net-(D2-Pad1)
- D2 pad 2: (no net) -> Net-(D1-Pad1)
- D20 pad 1: GND -> (no net)
- D20 pad 2: Net-(D19-Pad1) -> (no net)
- D20 pad 1: (no net) -> GND
- D20 pad 2: (no net) -> Net-(D19-Pad1)
- D21 pad 1: Net-(D21-Pad1) -> (no net)
- D21 pad 2: +12V -> (no net)
- D21 pad 1: (no net) -> Net-(D21-Pad1)
- D21 pad 2: (no net) -> +12V
- D22 pad 1: Net-(D22-Pad1) -> (no net)
- D22 pad 2: Net-(D21-Pad1) -> (no net)
- D22 pad 1: (no net) -> Net-(D22-Pad1)
- D22 pad 2: (no net) -> Net-(D21-Pad1)
- D23 pad 1: Net-(D23-Pad1) -> (no net)
- D23 pad 2: Net-(D22-Pad1) -> (no net)
- D23 pad 1: (no net) -> Net-(D23-Pad1)
- D23 pad 2: (no net) -> Net-(D22-Pad1)
- D24 pad 1: GND -> (no net)
- D24 pad 2: Net-(D23-Pad1) -> (no net)
- D24 pad 1: (no net) -> GND
- D24 pad 2: (no net) -> Net-(D23-Pad1)
- D25 pad 1: Net-(D25-Pad1) -> (no net)
- D25 pad 2: +12V -> (no net)
- D25 pad 1: (no net) -> Net-(D25-Pad1)
- D25 pad 2: (no net) -> +12V
- D26 pad 1: Net-(D26-Pad1) -> (no net)
- D26 pad 2: Net-(D25-Pad1) -> (no net)
- D26 pad 1: (no net) -> Net-(D26-Pad1)
- D26 pad 2: (no net) -> Net-(D25-Pad1)
- D27 pad 1: Net-(D27-Pad1) -> (no net)
- D27 pad 2: Net-(D26-Pad1) -> (no net)
- D27 pad 1: (no net) -> Net-(D27-Pad1)
- D27 pad 2: (no net) -> Net-(D26-Pad1)
- D28 pad 1: GND -> (no net)
- D28 pad 2: Net-(D27-Pad1) -> (no net)
- D28 pad 1: (no net) -> GND
- D28 pad 2: (no net) -> Net-(D27-Pad1)
- D29 pad 1: Net-(D29-Pad1) -> (no net)
- D29 pad 2: +12V -> (no net)
- D29 pad 1: (no net) -> Net-(D29-Pad1)
- D29 pad 2: (no net) -> +12V
- D3 pad 1: (no net) -> Net-(D3-Pad1)
- D3 pad 2: (no net) -> Net-(D2-Pad1)
- D30 pad 1: Net-(D30-Pad1) -> (no net)
- D30 pad 2: Net-(D29-Pad1) -> (no net)
- D30 pad 1: (no net) -> Net-(D30-Pad1)
- D30 pad 2: (no net) -> Net-(D29-Pad1)
- D31 pad 1: Net-(D31-Pad1) -> (no net)
- D31 pad 2: Net-(D30-Pad1) -> (no net)
- D31 pad 1: (no net) -> Net-(D31-Pad1)
- D31 pad 2: (no net) -> Net-(D30-Pad1)
- D32 pad 1: GND -> (no net)
- D32 pad 2: Net-(D31-Pad1) -> (no net)
- D32 pad 1: (no net) -> GND
- D32 pad 2: (no net) -> Net-(D31-Pad1)
- D33 pad 1: Net-(D33-Pad1) -> (no net)
- D33 pad 2: +12V -> (no net)
- D33 pad 1: (no net) -> Net-(D33-Pad1)
- D33 pad 2: (no net) -> +12V
- D34 pad 1: Net-(D34-Pad1) -> (no net)
- D34 pad 2: Net-(D33-Pad1) -> (no net)
- D34 pad 1: (no net) -> Net-(D34-Pad1)
- D34 pad 2: (no net) -> Net-(D33-Pad1)
- D35 pad 1: Net-(D35-Pad1) -> (no net)
- D35 pad 2: Net-(D34-Pad1) -> (no net)
- D35 pad 1: (no net) -> Net-(D35-Pad1)
- D35 pad 2: (no net) -> Net-(D34-Pad1)
- D36 pad 1: GND -> (no net)
- D36 pad 2: Net-(D35-Pad1) -> (no net)
- D36 pad 1: (no net) -> GND
- D36 pad 2: (no net) -> Net-(D35-Pad1)
- D37 pad 1: Net-(D37-Pad1) -> (no net)
- D37 pad 2: +12V -> (no net)
- D37 pad 1: (no net) -> Net-(D37-Pad1)
- D37 pad 2: (no net) -> +12V
- D38 pad 1: Net-(D38-Pad1) -> (no net)
- D38 pad 2: Net-(D37-Pad1) -> (no net)
- D38 pad 1: (no net) -> Net-(D38-Pad1)
- D38 pad 2: (no net) -> Net-(D37-Pad1)
- D39 pad 1: Net-(D39-Pad1) -> (no net)
- D39 pad 2: Net-(D38-Pad1) -> (no net)
- D39 pad 1: (no net) -> Net-(D39-Pad1)
- D39 pad 2: (no net) -> Net-(D38-Pad1)
- D4 pad 1: (no net) -> GND
- D4 pad 2: (no net) -> Net-(D3-Pad1)
- D40 pad 1: GND -> (no net)
- D40 pad 2: Net-(D39-Pad1) -> (no net)
- D40 pad 1: (no net) -> GND
- D40 pad 2: (no net) -> Net-(D39-Pad1)
- D41 pad 1: Net-(D41-Pad1) -> (no net)
- D41 pad 2: +12V -> (no net)
- D41 pad 1: (no net) -> Net-(D41-Pad1)
- D41 pad 2: (no net) -> +12V
- D42 pad 1: Net-(D42-Pad1) -> (no net)
- D42 pad 2: Net-(D41-Pad1) -> (no net)
- D42 pad 1: (no net) -> Net-(D42-Pad1)
- D42 pad 2: (no net) -> Net-(D41-Pad1)
- D43 pad 1: Net-(D43-Pad1) -> (no net)
- D43 pad 2: Net-(D42-Pad1) -> (no net)
- D43 pad 1: (no net) -> Net-(D43-Pad1)
- D43 pad 2: (no net) -> Net-(D42-Pad1)
- D44 pad 1: GND -> (no net)
- D44 pad 2: Net-(D43-Pad1) -> (no net)
- D44 pad 1: (no net) -> GND
- D44 pad 2: (no net) -> Net-(D43-Pad1)
- D45 pad 1: Net-(D45-Pad1) -> (no net)
- D45 pad 2: +12V -> (no net)
- D45 pad 1: (no net) -> Net-(D45-Pad1)
- D45 pad 2: (no net) -> +12V
- D46 pad 1: Net-(D46-Pad1) -> (no net)
- D46 pad 2: Net-(D45-Pad1) -> (no net)
- D46 pad 1: (no net) -> Net-(D46-Pad1)
- D46 pad 2: (no net) -> Net-(D45-Pad1)
- D47 pad 1: Net-(D47-Pad1) -> (no net)
- D47 pad 2: Net-(D46-Pad1) -> (no net)
- D47 pad 1: (no net) -> Net-(D47-Pad1)
- D47 pad 2: (no net) -> Net-(D46-Pad1)
- D48 pad 1: GND -> (no net)
- D48 pad 2: Net-(D47-Pad1) -> (no net)
- D48 pad 1: (no net) -> GND
- D48 pad 2: (no net) -> Net-(D47-Pad1)
- D49 pad 1: Net-(D49-Pad1) -> (no net)
- D49 pad 2: +12V -> (no net)
- D49 pad 1: (no net) -> Net-(D49-Pad1)
- D49 pad 2: (no net) -> +12V
- D5 pad 1: Net-(D5-Pad1) -> (no net)
- D5 pad 2: +12V -> (no net)
- D5 pad 1: (no net) -> Net-(D5-Pad1)
- D5 pad 2: (no net) -> +12V
- D50 pad 1: Net-(D50-Pad1) -> (no net)
- D50 pad 2: Net-(D49-Pad1) -> (no net)
- D50 pad 1: (no net) -> Net-(D50-Pad1)
- D50 pad 2: (no net) -> Net-(D49-Pad1)
- D51 pad 1: Net-(D51-Pad1) -> (no net)
- D51 pad 2: Net-(D50-Pad1) -> (no net)
- D51 pad 1: (no net) -> Net-(D51-Pad1)
- D51 pad 2: (no net) -> Net-(D50-Pad1)
- D52 pad 1: GND -> (no net)
- D52 pad 2: Net-(D51-Pad1) -> (no net)
- D52 pad 1: (no net) -> GND
- D52 pad 2: (no net) -> Net-(D51-Pad1)
- D53 pad 1: Net-(D53-Pad1) -> (no net)
- D53 pad 2: +12V -> (no net)
- D53 pad 1: (no net) -> Net-(D53-Pad1)
- D53 pad 2: (no net) -> +12V
- D54 pad 1: Net-(D54-Pad1) -> (no net)
- D54 pad 2: Net-(D53-Pad1) -> (no net)
- D54 pad 1: (no net) -> Net-(D54-Pad1)
- D54 pad 2: (no net) -> Net-(D53-Pad1)
- D55 pad 1: Net-(D55-Pad1) -> (no net)
- D55 pad 2: Net-(D54-Pad1) -> (no net)
- D55 pad 1: (no net) -> Net-(D55-Pad1)
- D55 pad 2: (no net) -> Net-(D54-Pad1)
- D56 pad 1: GND -> (no net)
- D56 pad 2: Net-(D55-Pad1) -> (no net)
- D56 pad 1: (no net) -> GND
- D56 pad 2: (no net) -> Net-(D55-Pad1)
- D57 pad 1: Net-(D57-Pad1) -> (no net)
- D57 pad 2: +12V -> (no net)
- D57 pad 1: (no net) -> Net-(D57-Pad1)
- D57 pad 2: (no net) -> +12V
- D58 pad 1: Net-(D58-Pad1) -> (no net)
- D58 pad 2: Net-(D57-Pad1) -> (no net)
- D58 pad 1: (no net) -> Net-(D58-Pad1)
- D58 pad 2: (no net) -> Net-(D57-Pad1)
- D59 pad 1: Net-(D59-Pad1) -> (no net)
- D59 pad 2: Net-(D58-Pad1) -> (no net)
- D59 pad 1: (no net) -> Net-(D59-Pad1)
- D59 pad 2: (no net) -> Net-(D58-Pad1)
- D6 pad 1: Net-(D6-Pad1) -> (no net)
- D6 pad 2: Net-(D5-Pad1) -> (no net)
- D6 pad 1: (no net) -> Net-(D6-Pad1)
- D6 pad 2: (no net) -> Net-(D5-Pad1)
- D60 pad 1: GND -> (no net)
- D60 pad 2: Net-(D59-Pad1) -> (no net)
- D60 pad 1: (no net) -> GND
- D60 pad 2: (no net) -> Net-(D59-Pad1)
- D61 pad 1: Net-(D61-Pad1) -> (no net)
- D61 pad 2: +12V -> (no net)
- D61 pad 1: (no net) -> Net-(D61-Pad1)
- D61 pad 2: (no net) -> +12V
- D7 pad 1: Net-(D7-Pad1) -> (no net)
- D7 pad 2: Net-(D6-Pad1) -> (no net)
- D7 pad 1: (no net) -> Net-(D7-Pad1)
- D7 pad 2: (no net) -> Net-(D6-Pad1)
- D8 pad 1: GND -> (no net)
- D8 pad 2: Net-(D7-Pad1) -> (no net)
- D8 pad 1: (no net) -> GND
- D8 pad 2: (no net) -> Net-(D7-Pad1)
- D9 pad 1: Net-(D10-Pad2) -> (no net)
- D9 pad 2: +12V -> (no net)
- D9 pad 1: (no net) -> Net-(D10-Pad2)
- D9 pad 2: (no net) -> +12V
Routing:
- net GND: track 0.00 -> 1153.9 mm, vias 0 -> 2
- net +12V: track 0.00 -> 833.0 mm, vias 0 -> 2
- net Net-(D11-Pad1): track 0.00 -> 31.2 mm
- net Net-(D46-Pad1): track 0.00 -> 30.5 mm
- net Net-(D47-Pad1): track 0.00 -> 30.4 mm
- net Net-(D45-Pad1): track 0.00 -> 30.4 mm
- net Net-(D3-Pad1): track 0.00 -> 29.9 mm
- net Net-(D25-Pad1): track 0.00 -> 29.3 mm
- net Net-(D27-Pad1): track 0.00 -> 29.0 mm
- net Net-(D26-Pad1): track 0.00 -> 27.9 mm
- net Net-(D10-Pad1): track 0.00 -> 27.1 mm
- net Net-(D49-Pad1): track 0.00 -> 26.8 mm
- net Net-(D13-Pad1): track 0.00 -> 26.6 mm
- net Net-(D37-Pad1): track 0.00 -> 26.0 mm
- net Net-(D19-Pad1): track 0.00 -> 25.1 mm
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Other:
- net class Default: clearance 0.2 -> 0.5
- rule trace_clearance: 0.2 -> 0.5

Commit message: add files to toggle switch, add new componnents to plc
Parts:
- added D62: 1N4007, Diode_THT:D_DO-41_SOD81_P10.16mm_Horizontal, F.Cu at (607.2, -159.0)
- added D62: 1N4007, Diode_THT:D_DO-41_SOD81_P10.16mm_Horizontal, F.Cu at (482.0, 112.7)
- added J1: Screw_Terminal_01x03, Connector_Phoenix_MSTB:PhoenixContact_MSTBVA_2,5_3-G-5,08_1x03_P5.08mm_Vertical, F.Cu at (609.9, -165.9)
- added J1: Screw_Terminal_01x03, Connector_Phoenix_MSTB:PhoenixContact_MSTBVA_2,5_3-G-5,08_1x03_P5.08mm_Vertical, B.Cu at (463.9, 112.6)
- moved D1 101.4 mm to (631.1, -321.9)
- moved D10 101.4 mm to (624.1, -303.9)
- moved D11 101.4 mm to (617.1, -303.9)
- moved D12 101.4 mm to (610.1, -303.9)
- moved D13 101.4 mm to (631.1, -294.9)
- moved D14 101.4 mm to (624.1, -294.9)
- moved D15 101.4 mm to (617.1, -294.9)
- moved D16 101.4 mm to (610.1, -294.9)
- moved D17 101.4 mm to (631.1, -285.9)
- moved D18 101.4 mm to (624.1, -285.9)
- moved D19 101.4 mm to (617.1, -285.9)
- moved D2 101.4 mm to (624.1, -321.9)
- moved D20 101.4 mm to (610.1, -285.9)
- moved D21 101.4 mm to (631.1, -276.9)
- moved D22 101.4 mm to (624.1, -276.9)
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Routing:
- net GND: track 1153.9 -> 1180.6 mm
- net Net-(D62-Pad1): track 0.00 -> 19.3 mm
- net +12V: track 833.0 -> 851.4 mm
