File: HARDWARE/EDA/KICAD/PLC/PLC.kicad_pcb (KiCad board)
At the start: 2 copper layers, 202 x 541.8 mm, 128 parts, among them J1 Screw_Terminal_01x03

Commit message: finished new schametic
Parts:
- moved D1 471.3 mm to (786.7, -242.9)
- moved D10 471.3 mm to (752.1, -262.9)
- moved D12 471.3 mm to (786.7, -282.9)
- moved D14 471.3 mm to (821.4, -262.9)
- moved D15 471.3 mm to (826.7, -242.9)
- moved D17 471.3 mm to (806.7, -208.2)
- moved D18 471.3 mm to (786.7, -202.9)
- moved D19 471.3 mm to (766.7, -208.3)
- moved D2 471.3 mm to (766.7, -242.9)
- moved D20 471.3 mm to (740.7, -204.3)
- moved D21 471.3 mm to (730.4, -222.4)
- moved D22 471.3 mm to (726.7, -242.9)
- moved D23 471.3 mm to (730.4, -263.4)
- moved D24 471.3 mm to (740.7, -281.4)
- moved D25 471.3 mm to (756.7, -294.9)
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Connections:
- D1 pad 1: Net-(D1-Pad1) -> (no net)
- D1 pad 2: +12V -> (no net)
- D10 pad 1: Net-(D10-Pad1) -> (no net)
- D10 pad 2: Net-(D10-Pad2) -> (no net)
- D11 pad 1: Net-(D11-Pad1) -> (no net)
- D11 pad 2: Net-(D10-Pad1) -> (no net)
- D12 pad 1: GND -> (no net)
- D12 pad 2: Net-(D11-Pad1) -> (no net)
- D13 pad 1: Net-(D13-Pad1) -> (no net)
- D13 pad 2: +12V -> (no net)
- D14 pad 1: Net-(D14-Pad1) -> (no net)
- D14 pad 2: Net-(D13-Pad1) -> (no net)
- D15 pad 1: Net-(D15-Pad1) -> (no net)
- D15 pad 2: Net-(D14-Pad1) -> (no net)
- D16 pad 1: GND -> (no net)
- D16 pad 2: Net-(D15-Pad1) -> (no net)
- D17 pad 1: Net-(D17-Pad1) -> (no net)
- D17 pad 2: +12V -> (no net)
- D18 pad 1: Net-(D18-Pad1) -> (no net)
- D18 pad 2: Net-(D17-Pad1) -> (no net)
- D19 pad 1: Net-(D19-Pad1) -> (no net)
- D19 pad 2: Net-(D18-Pad1) -> (no net)
- D2 pad 1: Net-(D2-Pad1) -> (no net)
- D2 pad 2: Net-(D1-Pad1) -> (no net)
- D20 pad 1: GND -> (no net)
- D20 pad 2: Net-(D19-Pad1) -> (no net)
- D21 pad 1: Net-(D21-Pad1) -> (no net)
- D21 pad 2: +12V -> (no net)
- D22 pad 1: Net-(D22-Pad1) -> (no net)
- D22 pad 2: Net-(D21-Pad1) -> (no net)
- D23 pad 1: Net-(D23-Pad1) -> (no net)
- D23 pad 2: Net-(D22-Pad1) -> (no net)
- D24 pad 1: GND -> (no net)
- D24 pad 2: Net-(D23-Pad1) -> (no net)
- D25 pad 1: Net-(D25-Pad1) -> (no net)
- D25 pad 2: +12V -> (no net)
- D26 pad 1: Net-(D26-Pad1) -> (no net)
- D26 pad 2: Net-(D25-Pad1) -> (no net)
- D27 pad 1: Net-(D27-Pad1) -> (no net)
- D27 pad 2: Net-(D26-Pad1) -> (no net)
- D28 pad 1: GND -> (no net)
- D28 pad 2: Net-(D27-Pad1) -> (no net)
- D29 pad 1: Net-(D29-Pad1) -> (no net)
- D29 pad 2: +12V -> (no net)
- D3 pad 1: Net-(D3-Pad1) -> (no net)
- D3 pad 2: Net-(D2-Pad1) -> (no net)
- D30 pad 1: Net-(D30-Pad1) -> (no net)
- D30 pad 2: Net-(D29-Pad1) -> (no net)
- D31 pad 1: Net-(D31-Pad1) -> (no net)
- D31 pad 2: Net-(D30-Pad1) -> (no net)
- D32 pad 1: GND -> (no net)
- D32 pad 2: Net-(D31-Pad1) -> (no net)
- D33 pad 1: Net-(D33-Pad1) -> (no net)
- D33 pad 2: +12V -> (no net)
- D34 pad 1: Net-(D34-Pad1) -> (no net)
- D34 pad 2: Net-(D33-Pad1) -> (no net)
- D35 pad 1: Net-(D35-Pad1) -> (no net)
- D35 pad 2: Net-(D34-Pad1) -> (no net)
- D36 pad 1: GND -> (no net)
- D36 pad 2: Net-(D35-Pad1) -> (no net)
- D37 pad 1: Net-(D37-Pad1) -> (no net)
- D37 pad 2: +12V -> (no net)
- D38 pad 1: Net-(D38-Pad1) -> (no net)
- D38 pad 2: Net-(D37-Pad1) -> (no net)
- D39 pad 1: Net-(D39-Pad1) -> (no net)
- D39 pad 2: Net-(D38-Pad1) -> (no net)
- D4 pad 1: GND -> (no net)
- D4 pad 2: Net-(D3-Pad1) -> (no net)
- D40 pad 1: GND -> (no net)
- D40 pad 2: Net-(D39-Pad1) -> (no net)
- D41 pad 1: Net-(D41-Pad1) -> (no net)
- D41 pad 2: +12V -> (no net)
- D42 pad 1: Net-(D42-Pad1) -> (no net)
- D42 pad 2: Net-(D41-Pad1) -> (no net)
- D43 pad 1: Net-(D43-Pad1) -> (no net)
- D43 pad 2: Net-(D42-Pad1) -> (no net)
- D44 pad 1: GND -> (no net)
- D44 pad 2: Net-(D43-Pad1) -> (no net)
- D45 pad 1: Net-(D45-Pad1) -> (no net)
- D45 pad 2: +12V -> (no net)
- D46 pad 1: Net-(D46-Pad1) -> (no net)
- D46 pad 2: Net-(D45-Pad1) -> (no net)
- D47 pad 1: Net-(D47-Pad1) -> (no net)
- D47 pad 2: Net-(D46-Pad1) -> (no net)
- D48 pad 1: GND -> (no net)
- D48 pad 2: Net-(D47-Pad1) -> (no net)
- D49 pad 1: Net-(D49-Pad1) -> (no net)
- D49 pad 2: +12V -> (no net)
- D5 pad 1: Net-(D5-Pad1) -> (no net)
- D5 pad 2: +12V -> (no net)
- D50 pad 1: Net-(D50-Pad1) -> (no net)
- D50 pad 2: Net-(D49-Pad1) -> (no net)
- D51 pad 1: Net-(D51-Pad1) -> (no net)
- D51 pad 2: Net-(D50-Pad1) -> (no net)
- D52 pad 1: GND -> (no net)
- D52 pad 2: Net-(D51-Pad1) -> (no net)
- D53 pad 1: Net-(D53-Pad1) -> (no net)
- D53 pad 2: +12V -> (no net)
- D54 pad 1: Net-(D54-Pad1) -> (no net)
- D54 pad 2: Net-(D53-Pad1) -> (no net)
- D55 pad 1: Net-(D55-Pad1) -> (no net)
- D55 pad 2: Net-(D54-Pad1) -> (no net)
- D56 pad 1: GND -> (no net)
- D56 pad 2: Net-(D55-Pad1) -> (no net)
- D57 pad 1: Net-(D57-Pad1) -> (no net)
- D57 pad 2: +12V -> (no net)
- D58 pad 1: Net-(D58-Pad1) -> (no net)
- D58 pad 2: Net-(D57-Pad1) -> (no net)
- D59 pad 1: Net-(D59-Pad1) -> (no net)
- D59 pad 2: Net-(D58-Pad1) -> (no net)
- D6 pad 1: Net-(D6-Pad1) -> (no net)
- D6 pad 2: Net-(D5-Pad1) -> (no net)
- D60 pad 1: GND -> (no net)
- D60 pad 2: Net-(D59-Pad1) -> (no net)
- D61 pad 1: Net-(D61-Pad1) -> (no net)
- D61 pad 2: +12V -> (no net)
- D62 pad 1: Net-(D62-Pad1) -> (no net)
- D62 pad 2: +12V -> (no net)
- D7 pad 1: Net-(D7-Pad1) -> (no net)
- D7 pad 2: Net-(D6-Pad1) -> (no net)
- D8 pad 1: GND -> (no net)
- D8 pad 2: Net-(D7-Pad1) -> (no net)
- D9 pad 1: Net-(D10-Pad2) -> (no net)
- D9 pad 2: +12V -> (no net)
- J1 pad 1: GND -> (no net)
- J1 pad 2: Net-(D62-Pad1) -> (no net)
- J1 pad 3: +12V -> (no net)
- R1 pad 1: GND -> (no net)
- R1 pad 2: Net-(D61-Pad1) -> (no net)
Routing:
- net (no net): track 0.00 -> 3109.2 mm, vias 0 -> 4
- net GND: track 1180.6 -> 0.00 mm, vias 2 -> 0
- net +12V: track 851.4 -> 0.00 mm, vias 2 -> 0
- net Net-(D11-Pad1): track 31.2 -> 0.00 mm
- net Net-(D46-Pad1): track 30.5 -> 0.00 mm
- net Net-(D47-Pad1): track 30.4 -> 0.00 mm
- net Net-(D45-Pad1): track 30.4 -> 0.00 mm
- net Net-(D3-Pad1): track 29.9 -> 0.00 mm
- net Net-(D25-Pad1): track 29.3 -> 0.00 mm
- net Net-(D27-Pad1): track 29.0 -> 0.00 mm
- net Net-(D26-Pad1): track 27.9 -> 0.00 mm
- net Net-(D10-Pad1): track 27.1 -> 0.00 mm
- net Net-(D49-Pad1): track 26.8 -> 0.00 mm
- net Net-(D13-Pad1): track 26.6 -> 0.00 mm
- net Net-(D37-Pad1): track 26.0 -> 0.00 mm
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Other:
- board size 202 x 541.8 mm -> 519 x 546.9 mm

Commit message: remix project
Parts:
- removed the D1 at (786.7, -242.9)
- removed the D10 at (752.1, -262.9)
- removed the D11 at (766.8, -277.5)
- removed the D12 at (786.7, -282.9)
- removed the D13 at (806.8, -277.5)
- removed the D14 at (821.4, -262.9)
- removed the D15 at (826.7, -242.9)
- removed the D16 at (821.3, -222.9)
- removed the D17 at (806.7, -208.2)
- removed the D18 at (786.7, -202.9)
- removed the D19 at (766.7, -208.3)
- removed the D2 at (766.7, -242.9)
- removed the D20 at (740.7, -204.3)
- removed the D21 at (730.4, -222.4)
- removed the D21 at (631.1, -276.9)
- removed the D22 at (726.7, -242.9)
- removed the D23 at (730.4, -263.4)
- removed the D24 at (740.7, -281.4)
- removed the D25 at (756.7, -294.9)
- removed the D25 at (631.1, -267.9)
- removed the D26 at (776.3, -302.0)
- removed the D27 at (797.1, -302.0)
- removed the D28 at (816.7, -294.9)
- removed the D29 at (832.7, -281.5)
- removed the D3 at (776.8, -260.2)
- removed the D30 at (843.1, -263.4)
- removed the D31 at (846.7, -242.9)
- removed the D32 at (843.1, -222.3)
- removed the D33 at (832.7, -204.3)
- removed the D34 at (816.7, -190.9)
- removed the D35 at (797.1, -183.8)
- removed the D36 at (776.3, -183.8)
- removed the D37 at (756.7, -190.9)
- removed the D38 at (730.1, -186.3)
- removed the D39 at (717.4, -202.9)
- removed the D4 at (796.7, -260.2)
- removed the D40 at (709.5, -222.2)
- removed the D41 at (706.7, -242.9)
- removed the D42 at (709.4, -263.6)
- removed the D43 at (717.5, -282.9)
- removed the D44 at (730.2, -299.5)
- removed the D45 at (746.7, -312.1)
- removed the D46 at (766.0, -320.2)
- removed the D47 at (786.7, -322.9)
- removed the D48 at (807.5, -320.2)
- removed the D49 at (826.7, -312.2)
- removed the D5 at (806.7, -242.9)
- removed the D50 at (843.3, -299.5)
- removed the D51 at (856.0, -282.9)
- removed the D52 at (864.0, -263.6)
- removed the D53 at (866.7, -242.9)
- removed the D53 at (631.1, -204.9)
- removed the D54 at (864.0, -222.2)
- removed the D54 at (624.1, -204.9)
- removed the D55 at (856.0, -202.9)
- removed the D55 at (617.1, -204.9)
- removed the D56 at (843.3, -186.3)
- removed the D56 at (610.1, -204.9)
- removed the D57 at (826.7, -173.6)
- removed the D58 at (807.4, -165.7)
- removed the D59 at (786.7, -162.9)
- removed the D6 at (796.7, -225.5)
- removed the D60 at (766.0, -165.6)
- removed the D61 at (746.7, -173.6)
- removed the D62 at (801.0, -234.2)
- removed the D7 at (776.7, -225.5)
- removed the D8 at (752.1, -222.9)
- removed the D9 at (746.8, -242.9)
- removed the J1 at (782.9, -234.3)
- removed the R1 at (735.8, -173.7)
- removed the R1 at (618.5, -185.9)
- added C1: 16V 330uf, Capacitor_THT:CP_Radial_D8.0mm_P3.50mm, B.Cu at (115.8, 97.6)
- added D1: LED, LED_THT:LED_D5.0mm, F.Cu at (630.6, -321.1)
- added D1: LED, LED_THT:LED_D5.0mm, F.Cu at (812.0, -237.2)
- added D10: LED, LED_THT:LED_D5.0mm_IRBlack, F.Cu at (777.5, -257.2)
- added D10: LED, LED_THT:LED_D5.0mm_IRBlack, F.Cu at (623.6, -303.1)
- added D11: LED, LED_THT:LED_D5.0mm_IRBlack, F.Cu at (792.1, -271.9)
- added D11: LED, LED_THT:LED_D5.0mm_IRBlack, F.Cu at (616.6, -303.1)
- added D12: LED, LED_THT:LED_D5.0mm_IRBlack, F.Cu at (609.6, -303.1)
- added D12: LED, LED_THT:LED_D5.0mm_IRBlack, F.Cu at (812.0, -277.2)
- added D13: LED, LED_THT:LED_D5.0mm_IRGrey, F.Cu at (630.6, -294.1)
- added D13: LED, LED_THT:LED_D5.0mm_IRGrey, F.Cu at (832.1, -271.9)
- added D14: LED, LED_THT:LED_D5.0mm_IRGrey, F.Cu at (623.6, -294.1)
- added D14: LED, LED_THT:LED_D5.0mm_IRGrey, F.Cu at (846.8, -257.2)
- added D15: LED, LED_THT:LED_D5.0mm_IRGrey, F.Cu at (852.0, -237.2)
- added D15: LED, LED_THT:LED_D5.0mm_IRGrey, F.Cu at (616.6, -294.1)
- added D16: LED, LED_THT:LED_D5.0mm_IRGrey, F.Cu at (846.6, -217.2)
- added D16: LED, LED_THT:LED_D5.0mm_IRGrey, F.Cu at (609.6, -294.1)
- added D17: LED, LED_THT:LED_D5.0mm, F.Cu at (630.6, -285.1)
- added D17: LED, LED_THT:LED_D5.0mm, F.Cu at (832.0, -202.6)
- added D18: LED, LED_THT:LED_D5.0mm, F.Cu at (623.6, -285.1)
- added D18: LED, LED_THT:LED_D5.0mm, F.Cu at (812.0, -197.2)
- added D19: LED, LED_THT:LED_D5.0mm, F.Cu at (616.6, -285.1)
- added D19: LED, LED_THT:LED_D5.0mm, F.Cu at (792.0, -202.7)
- added D2: LED, LED_THT:LED_D5.0mm, F.Cu at (792.0, -237.2)
- added D2: LED, LED_THT:LED_D5.0mm, F.Cu at (623.6, -321.1)
- added D20: LED, LED_THT:LED_D5.0mm, F.Cu at (609.6, -285.1)
- added D20: LED, LED_THT:LED_D5.0mm, F.Cu at (766.0, -198.7)
- added D21: LED, LED_THT:LED_D5.0mm_Clear, F.Cu at (755.8, -216.8)
- added D21: LED, LED_THT:LED_D5.0mm_Clear, F.Cu at (630.6, -276.1)
- added D21: LED, LED_THT:LED_D5.0mm_Clear, F.Cu at (30.9, 104.0)
- added D22: LED, LED_THT:LED_D5.0mm_Clear, F.Cu at (752.0, -237.2)
- added D22: LED, LED_THT:LED_D5.0mm_Clear, F.Cu at (623.6, -276.1)
- added D23: LED, LED_THT:LED_D5.0mm_Clear, F.Cu at (616.6, -276.1)
- added D23: LED, LED_THT:LED_D5.0mm_Clear, F.Cu at (755.8, -257.8)
- added D24: LED, LED_THT:LED_D5.0mm_Clear, F.Cu at (766.0, -275.8)
- added D24: LED, LED_THT:LED_D5.0mm_Clear, F.Cu at (609.6, -276.1)
- added D25: LED, LED_THT:LED_D5.0mm_IRBlack, F.Cu at (630.6, -267.1)
- added D25: LED, LED_THT:LED_D5.0mm_IRBlack, F.Cu at (782.0, -289.2)
- added D25: LED, LED_THT:LED_D5.0mm_IRBlack, F.Cu at (81.0, 52.1)
- added D26: LED, LED_THT:LED_D5.0mm_IRBlack, F.Cu at (623.6, -267.1)
- added D26: LED, LED_THT:LED_D5.0mm_IRBlack, F.Cu at (801.6, -296.4)
- added D27: LED, LED_THT:LED_D5.0mm_IRBlack, F.Cu at (616.6, -267.1)
- added D27: LED, LED_THT:LED_D5.0mm_IRBlack, F.Cu at (822.5, -296.4)
- added D28: LED, LED_THT:LED_D5.0mm_IRBlack, F.Cu at (842.0, -289.2)
- added D28: LED, LED_THT:LED_D5.0mm_IRBlack, F.Cu at (609.6, -267.1)
- added D29: LED, LED_THT:LED_D5.0mm_IRGrey, F.Cu at (858.0, -275.9)
- added D29: LED, LED_THT:LED_D5.0mm_IRGrey, F.Cu at (630.6, -258.1)
- added D3: LED, LED_THT:LED_D5.0mm, F.Cu at (616.6, -321.1)
- added D3: LED, LED_THT:LED_D5.0mm, F.Cu at (802.1, -254.6)
- added D30: LED, LED_THT:LED_D5.0mm_IRGrey, F.Cu at (868.5, -257.8)
- added D30: LED, LED_THT:LED_D5.0mm_IRGrey, F.Cu at (623.6, -258.1)
- added D31: LED, LED_THT:LED_D5.0mm_IRGrey, F.Cu at (872.0, -237.2)
- added D31: LED, LED_THT:LED_D5.0mm_IRGrey, F.Cu at (616.6, -258.1)
- added D32: LED, LED_THT:LED_D5.0mm_IRGrey, F.Cu at (868.5, -216.7)
- added D32: LED, LED_THT:LED_D5.0mm_IRGrey, F.Cu at (609.6, -258.1)
- added D33: LED, LED_THT:LED_D5.0mm, F.Cu at (630.6, -249.2)
- added D33: LED, LED_THT:LED_D5.0mm, F.Cu at (858.0, -198.7)
- added D34: LED, LED_THT:LED_D5.0mm, F.Cu at (623.6, -249.2)
- added D34: LED, LED_THT:LED_D5.0mm, F.Cu at (842.0, -185.2)
- added D35: LED, LED_THT:LED_D5.0mm, F.Cu at (616.6, -249.2)
- added D35: LED, LED_THT:LED_D5.0mm, F.Cu at (822.5, -178.2)
- added D36: LED, LED_THT:LED_D5.0mm, F.Cu at (609.6, -249.2)
- added D36: LED, LED_THT:LED_D5.0mm, F.Cu at (801.6, -178.2)
- added D37: LED, LED_THT:LED_D5.0mm_Clear, F.Cu at (782.0, -185.2)
- added D37: LED, LED_THT:LED_D5.0mm_Clear, F.Cu at (630.6, -240.2)
- added D38: LED, LED_THT:LED_D5.0mm_Clear, F.Cu at (755.5, -180.7)
- added D38: LED, LED_THT:LED_D5.0mm_Clear, F.Cu at (623.6, -240.2)
- added D39: LED, LED_THT:LED_D5.0mm_Clear, F.Cu at (616.6, -240.2)
- added D39: LED, LED_THT:LED_D5.0mm_Clear, F.Cu at (742.8, -197.2)
- added D4: LED, LED_THT:LED_D5.0mm, F.Cu at (822.0, -254.6)
- added D4: LED, LED_THT:LED_D5.0mm, F.Cu at (609.6, -321.1)
- added D40: LED, LED_THT:LED_D5.0mm_Clear, F.Cu at (734.9, -216.6)
- added D40: LED, LED_THT:LED_D5.0mm_Clear, F.Cu at (609.6, -240.2)
- added D41: LED, LED_THT:LED_D5.0mm_IRBlack, F.Cu at (630.6, -231.2)
- added D41: LED, LED_THT:LED_D5.0mm_IRBlack, F.Cu at (732.0, -237.2)
- added D42: LED, LED_THT:LED_D5.0mm_IRBlack, F.Cu at (623.6, -231.2)
- added D42: LED, LED_THT:LED_D5.0mm_IRBlack, F.Cu at (734.8, -257.9)
- added D43: LED, LED_THT:LED_D5.0mm_IRBlack, F.Cu at (742.9, -277.2)
- added D43: LED, LED_THT:LED_D5.0mm_IRBlack, F.Cu at (616.6, -231.2)
- added D44: LED, LED_THT:LED_D5.0mm_IRBlack, F.Cu at (755.5, -293.9)
- added D44: LED, LED_THT:LED_D5.0mm_IRBlack, F.Cu at (609.6, -231.2)
- added D45: LED, LED_THT:LED_D5.0mm_IRGrey, F.Cu at (630.6, -222.2)
- added D45: LED, LED_THT:LED_D5.0mm_IRGrey, F.Cu at (772.0, -306.4)
- added D46: LED, LED_THT:LED_D5.0mm_IRGrey, F.Cu at (791.4, -314.6)
- added D46: LED, LED_THT:LED_D5.0mm_IRGrey, F.Cu at (623.6, -222.2)
- added D47: LED, LED_THT:LED_D5.0mm_IRGrey, F.Cu at (616.6, -222.2)
- added D47: LED, LED_THT:LED_D5.0mm_IRGrey, F.Cu at (812.0, -317.2)
- added D48: LED, LED_THT:LED_D5.0mm_IRGrey, F.Cu at (832.9, -314.6)
- added D48: LED, LED_THT:LED_D5.0mm_IRGrey, F.Cu at (609.6, -222.2)
- added D49: LED, LED_THT:LED_D5.0mm, F.Cu at (852.0, -306.6)
- added D49: LED, LED_THT:LED_D5.0mm, F.Cu at (630.6, -213.2)
- added D5: LED, LED_THT:LED_D5.0mm_Clear, F.Cu at (630.6, -312.1)
- added D5: LED, LED_THT:LED_D5.0mm_Clear, F.Cu at (832.0, -237.2)
- added D50: LED, LED_THT:LED_D5.0mm, F.Cu at (868.6, -293.9)
- added D50: LED, LED_THT:LED_D5.0mm, F.Cu at (623.6, -213.2)
- added D51: LED, LED_THT:LED_D5.0mm, F.Cu at (881.4, -277.2)
- added D51: LED, LED_THT:LED_D5.0mm, F.Cu at (616.6, -213.2)
- added D52: LED, LED_THT:LED_D5.0mm, F.Cu at (889.4, -257.9)
- added D52: LED, LED_THT:LED_D5.0mm, F.Cu at (609.6, -213.2)
- added D53: LED, LED_THT:LED_D5.0mm_Clear, F.Cu at (892.0, -237.2)
- added D53: LED, LED_THT:LED_D5.0mm_Clear, F.Cu at (630.6, -204.2)
- added D53: LED, LED_THT:LED_D5.0mm_Clear, F.Cu at (71.0, 104.0)
- added D54: LED, LED_THT:LED_D5.0mm_Clear, F.Cu at (623.6, -204.2)
- added D54: LED, LED_THT:LED_D5.0mm_Clear, F.Cu at (889.3, -216.6)
- added D54: LED, LED_THT:LED_D5.0mm_Clear, F.Cu at (76.3, 84.0)
- added D55: LED, LED_THT:LED_D5.0mm_Clear, F.Cu at (881.4, -197.2)
- added D55: LED, LED_THT:LED_D5.0mm_Clear, F.Cu at (616.6, -204.2)
- added D55: LED, LED_THT:LED_D5.0mm_Clear, F.Cu at (100.9, 86.7)
- added D56: LED, LED_THT:LED_D5.0mm_Clear, F.Cu at (609.6, -204.2)
- added D56: LED, LED_THT:LED_D5.0mm_Clear, F.Cu at (868.6, -180.7)
- added D56: LED, LED_THT:LED_D5.0mm_Clear, F.Cu at (120.9, 86.7)
- added D57: LED, LED_THT:LED_D5.0mm_IRBlack, F.Cu at (852.0, -167.9)
- added D57: LED, LED_THT:LED_D5.0mm_IRBlack, F.Cu at (630.6, -195.2)
- added D58: LED, LED_THT:LED_D5.0mm_IRBlack, F.Cu at (832.8, -160.1)
- added D58: LED, LED_THT:LED_D5.0mm_IRBlack, F.Cu at (623.6, -195.2)
- added D59: LED, LED_THT:LED_D5.0mm_IRBlack, F.Cu at (616.6, -195.2)
- added D59: LED, LED_THT:LED_D5.0mm_IRBlack, F.Cu at (812.0, -157.2)
- added D6: LED, LED_THT:LED_D5.0mm_Clear, F.Cu at (822.0, -219.8)
- added D6: LED, LED_THT:LED_D5.0mm_Clear, F.Cu at (623.6, -312.1)
- added D60: LED, LED_THT:LED_D5.0mm_IRBlack, F.Cu at (609.6, -195.2)
- added D60: LED, LED_THT:LED_D5.0mm_IRBlack, F.Cu at (791.4, -159.9)
- added D61: LED, LED_THT:LED_D5.0mm_IRGrey, F.Cu at (772.0, -167.9)
- added D61: LED, LED_THT:LED_D5.0mm_IRGrey, F.Cu at (630.6, -185.2)
- added D62: 1N4007, Diode_THT:D_DO-41_SOD81_P10.16mm_Horizontal, F.Cu at (826.4, -228.6)
- added D62: 1N4007, Diode_THT:D_DO-41_SOD81_P10.16mm_Horizontal, F.Cu at (606.8, -158.2)
- added D63: FEEDBACK, LED_THT:LED_D5.0mm_IRGrey, F.Cu at (626.5, -132.7)
- added D63: FEEDBACK, LED_THT:LED_D5.0mm_IRGrey, F.Cu at (233.8, 104.6)
- added D64: 1N47xxA, Diode_THT:D_DO-41_SOD81_P10.16mm_Horizontal, F.Cu at (123.6, 105.7)
- added D7: LED, LED_THT:LED_D5.0mm_Clear, F.Cu at (802.0, -219.8)
- added D7: LED, LED_THT:LED_D5.0mm_Clear, F.Cu at (616.6, -312.1)
- added D8: LED, LED_THT:LED_D5.0mm_Clear, F.Cu at (777.5, -217.2)
- added D8: LED, LED_THT:LED_D5.0mm_Clear, F.Cu at (609.6, -312.1)
- added D9: LED, LED_THT:LED_D5.0mm_IRBlack, F.Cu at (630.6, -303.1)
- added D9: LED, LED_THT:LED_D5.0mm_IRBlack, F.Cu at (772.1, -237.2)
- added F1: Fuse 1A, Fuse:Fuseholder_Blade_Mini_Keystone_3568, F.Cu at (636.5, -151.9)
- added F1: Fuse 1A, Fuse:Fuseholder_Blade_Mini_Keystone_3568, B.Cu at (114.7, 116.0)
- added J1: Screw_Terminal_01x03, Connector_Phoenix_MSTB:PhoenixContact_MSTBVA_2,5_3-G-5,08_1x03_P5.08mm_Vertical, B.Cu at (808.2, -228.7)
- added J1: Screw_Terminal_01x03, Connector_Phoenix_MSTB:PhoenixContact_MSTBVA_2,5_3-G-5,08_1x03_P5.08mm_Vertical, F.Cu at (609.4, -165.2)
- added J2: FEEDBACK, Connector_PinSocket_2.54mm:PinSocket_1x02_P2.54mm_Vertical, F.Cu at (624.7, -126.5)
- added J2: FEEDBACK, Connector_PinSocket_2.54mm:PinSocket_1x02_P2.54mm_Vertical, B.Cu at (115.8, 90.9)
- added J3: FEEDBACK, Connector_PinHeader_2.54mm:PinHeader_1x02_P2.54mm_Vertical, F.Cu at (635.0, -139.1)
- added J3: FEEDBACK, Connector_PinHeader_2.54mm:PinHeader_1x02_P2.54mm_Vertical, F.Cu at (227.3, 102.4)
- added R1: 300 R, Resistor_THT:R_Axial_DIN0207_L6.3mm_D2.5mm_P7.62mm_Horizontal, F.Cu at (618.0, -185.2)
- added R1: 300 R, Resistor_THT:R_Axial_DIN0207_L6.3mm_D2.5mm_P7.62mm_Horizontal, F.Cu at (761.1, -168.1)
- added R1: 300 R, Resistor_THT:R_Axial_DIN0207_L6.3mm_D2.5mm_P7.62mm_Horizontal, F.Cu at (105.5, 96.3)
- added R2: 300R 1W, Resistor_THT:R_Axial_DIN0411_L9.9mm_D3.6mm_P15.24mm_Horizontal, F.Cu at (606.9, -138.8)
- added R2: R 2W, Resistor_THT:R_Axial_DIN0411_L9.9mm_D3.6mm_P15.24mm_Horizontal, F.Cu at (127.3, 93.7)
- added RV1: 14V, Varistor:RV_Disc_D7mm_W3.4mm_P5mm, F.Cu at (625.9, -139.6)
- added RV1: 14V, Varistor:RV_Disc_D7mm_W3.4mm_P5mm, F.Cu at (102.5, 107.1)
- added RV2: 14V, Varistor:RV_Disc_D7mm_W3.4mm_P5mm, F.Cu at (615.6, -134.4)
- added RV2: 14V, Varistor:RV_Disc_D7mm_W3.4mm_P5mm, F.Cu at (101.3, 103.0)
- added RV3: 14V, Varistor:RV_Disc_D7mm_W3.4mm_P5mm, F.Cu at (615.6, -129.4)
- added RV3: 14V, Varistor:RV_Disc_D7mm_W3.4mm_P5mm, F.Cu at (97.3, 103.0)
- added S1: 220/12 V, PLC_library:SW_100SP1T1B4M2QE, F.Cu at (609.6, -129.1)
- J1: value Screw_Terminal_01x03 -> pw_input; moved to B.Cu
- moved D17 724.3 mm to (70.9, 173.2)
- moved D18 723.9 mm to (54.4, 160.6)
- moved D19 718.3 mm to (41.6, 144.0)
- moved D20 707.8 mm to (33.6, 124.8)
- moved D16 705.0 mm to (90.2, 181.3)
- moved D15 696.8 mm to (111.0, 184.0)
- moved D22 691.7 mm to (33.6, 83.2)
- moved D14 685.0 mm to (131.7, 181.3)
- moved D37 678.3 mm to (81.0, 155.9)
- moved D38 678.0 mm to (65.0, 142.6)
- moved D39 670.8 mm to (54.6, 124.5)
- moved D13 670.7 mm to (150.9, 173.3)
- moved D23 668.8 mm to (41.6, 64.0)
- moved D1 664.1 mm to (70.9, 34.8)
- moved D41 657.2 mm to (54.5, 83.5)
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Connections:
- D1 pad 1: (no net) -> Net-(D1-Pad1)
- D1 pad 2: (no net) -> PWR
- D10 pad 1: (no net) -> Net-(D10-Pad1)
- D10 pad 2: (no net) -> Net-(D10-Pad2)
- D11 pad 1: (no net) -> Net-(D11-Pad1)
- D11 pad 2: (no net) -> Net-(D10-Pad1)
- D12 pad 1: (no net) -> GND
- D12 pad 2: (no net) -> Net-(D11-Pad1)
- D13 pad 1: (no net) -> Net-(D13-Pad1)
- D13 pad 2: (no net) -> PWR
- D14 pad 1: (no net) -> Net-(D14-Pad1)
- D14 pad 2: (no net) -> Net-(D13-Pad1)
- D15 pad 1: (no net) -> Net-(D15-Pad1)
- D15 pad 2: (no net) -> Net-(D14-Pad1)
- D16 pad 1: (no net) -> GND
- D16 pad 2: (no net) -> Net-(D15-Pad1)
- D17 pad 1: (no net) -> Net-(D17-Pad1)
- D17 pad 2: (no net) -> PWR
- D18 pad 1: (no net) -> Net-(D18-Pad1)
- D18 pad 2: (no net) -> Net-(D17-Pad1)
- D19 pad 1: (no net) -> Net-(D19-Pad1)
- D19 pad 2: (no net) -> Net-(D18-Pad1)
- D2 pad 1: (no net) -> Net-(D2-Pad1)
- D2 pad 2: (no net) -> Net-(D1-Pad1)
- D20 pad 1: (no net) -> GND
- D20 pad 2: (no net) -> Net-(D19-Pad1)
- D22 pad 1: (no net) -> Net-(D22-Pad1)
- D22 pad 2: (no net) -> Net-(D21-Pad1)
- D23 pad 1: (no net) -> Net-(D23-Pad1)
- D23 pad 2: (no net) -> Net-(D22-Pad1)
- D24 pad 1: (no net) -> GND
- D24 pad 2: (no net) -> Net-(D23-Pad1)
- D26 pad 1: (no net) -> Net-(D26-Pad1)
- D26 pad 2: (no net) -> Net-(D25-Pad1)
- D27 pad 1: (no net) -> Net-(D27-Pad1)
- D27 pad 2: (no net) -> Net-(D26-Pad1)
- D28 pad 1: (no net) -> GND
- D28 pad 2: (no net) -> Net-(D27-Pad1)
- D29 pad 1: (no net) -> Net-(D29-Pad1)
- D29 pad 2: (no net) -> PWR
- D3 pad 1: (no net) -> Net-(D3-Pad1)
- D3 pad 2: (no net) -> Net-(D2-Pad1)
- D30 pad 1: (no net) -> Net-(D30-Pad1)
- D30 pad 2: (no net) -> Net-(D29-Pad1)
- D31 pad 1: (no net) -> Net-(D31-Pad1)
- D31 pad 2: (no net) -> Net-(D30-Pad1)
- D32 pad 1: (no net) -> GND
- D32 pad 2: (no net) -> Net-(D31-Pad1)
- D33 pad 1: (no net) -> Net-(D33-Pad1)
- D33 pad 2: (no net) -> PWR
- D34 pad 1: (no net) -> Net-(D34-Pad1)
- D34 pad 2: (no net) -> Net-(D33-Pad1)
- D35 pad 1: (no net) -> Net-(D35-Pad1)
- D35 pad 2: (no net) -> Net-(D34-Pad1)
- D36 pad 1: (no net) -> GND
- D36 pad 2: (no net) -> Net-(D35-Pad1)
- D37 pad 1: (no net) -> Net-(D37-Pad1)
- D37 pad 2: (no net) -> PWR
- D38 pad 1: (no net) -> Net-(D38-Pad1)
- D38 pad 2: (no net) -> Net-(D37-Pad1)
- D39 pad 1: (no net) -> Net-(D39-Pad1)
- D39 pad 2: (no net) -> Net-(D38-Pad1)
- D4 pad 1: (no net) -> GND
- D4 pad 2: (no net) -> Net-(D3-Pad1)
- D40 pad 1: (no net) -> GND
- D40 pad 2: (no net) -> Net-(D39-Pad1)
- D41 pad 1: (no net) -> Net-(D41-Pad1)
- D41 pad 2: (no net) -> PWR
- D42 pad 1: (no net) -> Net-(D42-Pad1)
- D42 pad 2: (no net) -> Net-(D41-Pad1)
- D43 pad 1: (no net) -> Net-(D43-Pad1)
- D43 pad 2: (no net) -> Net-(D42-Pad1)
- D44 pad 1: (no net) -> GND
- D44 pad 2: (no net) -> Net-(D43-Pad1)
- D45 pad 1: (no net) -> Net-(D45-Pad1)
- D45 pad 2: (no net) -> PWR
- D46 pad 1: (no net) -> Net-(D46-Pad1)
- D46 pad 2: (no net) -> Net-(D45-Pad1)
- D47 pad 1: (no net) -> Net-(D47-Pad1)
- D47 pad 2: (no net) -> Net-(D46-Pad1)
- D48 pad 1: (no net) -> GND
- D48 pad 2: (no net) -> Net-(D47-Pad1)
- D49 pad 1: (no net) -> Net-(D49-Pad1)
- D49 pad 2: (no net) -> PWR
- D5 pad 1: (no net) -> Net-(D5-Pad1)
- D5 pad 2: (no net) -> PWR
- D50 pad 1: (no net) -> Net-(D50-Pad1)
- D50 pad 2: (no net) -> Net-(D49-Pad1)
- D51 pad 1: (no net) -> Net-(D51-Pad1)
- D51 pad 2: (no net) -> Net-(D50-Pad1)
- D52 pad 1: (no net) -> GND
- D52 pad 2: (no net) -> Net-(D51-Pad1)
- D57 pad 1: (no net) -> Net-(D57-Pad1)
- D57 pad 2: (no net) -> PWR
- D58 pad 1: (no net) -> Net-(D58-Pad1)
- D58 pad 2: (no net) -> Net-(D57-Pad1)
- D59 pad 1: (no net) -> Net-(D59-Pad1)
- D59 pad 2: (no net) -> Net-(D58-Pad1)
- D6 pad 1: (no net) -> Net-(D6-Pad1)
- D6 pad 2: (no net) -> Net-(D5-Pad1)
- D60 pad 1: (no net) -> GND
- D60 pad 2: (no net) -> Net-(D59-Pad1)
- D61 pad 1: (no net) -> Net-(D61-Pad1)
- D61 pad 2: (no net) -> PWR
- D62 pad 1: (no net) -> Net-(D62-Pad1)
- D62 pad 2: (no net) -> Net-(C1-Pad1)
- D7 pad 1: (no net) -> Net-(D7-Pad1)
- D7 pad 2: (no net) -> Net-(D6-Pad1)
- D8 pad 1: (no net) -> GND
- D8 pad 2: (no net) -> Net-(D7-Pad1)
- D9 pad 1: (no net) -> Net-(D10-Pad2)
- D9 pad 2: (no net) -> PWR
- J1 pad 1: (no net) -> GND
- J1 pad 2: (no net) -> Net-(D62-Pad1)
- J1 pad 3: (no net) -> Net-(F1-Pad1)
Routing:
- net PWR: track 0.00 -> 824.3 mm
- net GND: track 0.00 -> 686.9 mm
- net Net-(C1-Pad1): track 0.00 -> 60.1 mm
- net Net-(D42-Pad1): track 0.00 -> 37.8 mm
- net Net-(D53-Pad1): track 0.00 -> 35.6 mm
- net Net-(D54-Pad1): track 0.00 -> 35.4 mm
- net Net-(D25-Pad1): track 0.00 -> 35.0 mm
- net Net-(D41-Pad1): track 0.00 -> 32.9 mm
- net Net-(D5-Pad1): track 0.00 -> 32.6 mm
- net Net-(D3-Pad1): track 0.00 -> 32.1 mm
- net Net-(D27-Pad1): track 0.00 -> 31.9 mm
- net Net-(D55-Pad1): track 0.00 -> 31.8 mm
- net Net-(D2-Pad1): track 0.00 -> 31.2 mm
- net Net-(D43-Pad1): track 0.00 -> 30.8 mm
- net Net-(D26-Pad1): track 0.00 -> 28.5 mm
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Other:
- board size 519 x 546.9 mm -> 901.1 x 541.8 mm
- net class Default: clearance 0.5 -> 0.25
- rule trace_clearance: 0.5 -> 0.25
